Commit message: first aproach to making the gripper

File: models/mbzirc/geometry.xacro (robot description, xacro)
@@ -75,5 +75,5 @@
     <origin xyz="0 0.24 -0.24" rpy="0 1.57 0" />
   </xacro:camera_macro>
-  <!-- Magnetic gripper -->
+  <!-- Magnetic gripper
   <link name="magnetic_gripper">
     <inertial>
@@ -95,4 +95,5 @@
     <limit effort="0" lower="0" upper="0" velocity="0"/>
   </joint>
+  -->
   <!-- Instantiate rotors -->
   <xacro:vertical_rotor

File: models/mbzirc/model.xacro (robot description, xacro)
@@ -16,4 +16,11 @@
   <!-- Instantiate mbzirc "mechanics" -->
   <xacro:include filename="$(find delivery_uav)/models/mbzirc/geometry.xacro" />
+  <!-- Include gripper -->
+  <xacro:include filename="$(find delivery_uav)/models/mbzirc/simple_gripper.xacro" />
+  <!-- Join the uav to the gripper-->
+  <joint name="arm_gripper_joint" type="fixed">
+    <parent link="base_link"/>
+    <child link="gripper_palm"/>
+  </joint>
   <xacro:if value="$(arg enable_gps_plugin)">
     <!-- Instantiate gps plugin. -->
