Commit message: changes in inertia values for the gripper

File: models/mbzirc/lidar.xacro (robot description, xacro)
@@ -1,24 +1,24 @@
 <?xml version="1.0"?>
 <robot xmlns:xacro="http://ros.org/wiki/xacro">
-    <!-- propiedades del gripper -->
+    <!-- propiedades del lidar -->
     <xacro:property name="lid_radius" value="0.04267" />
     <xacro:property name="lid_length" value="0.05867" />
-    <!-- descripcion de los links del gripper-->
-    <link name="gripper_palm">
+    <!-- descripcion de los links del lidar-->
+    <link name="lidar_base">
         <collision>
-            <origin xyz="${basex} 0 ${basez}" rpy="0 0 0"/>
+            <origin xyz="0 0 ${0.5 * lid_length}" rpy="0 0 0"/>
             <geometry>
-                <box size="${defwidth} ${palm_length} ${defwidth}"/>
+                <<cylinder radius="${lid_radius}" length="${lid_length}"/>
             </geometry>
         </collision>
         <visual>
-            <origin xyz="${basex} 0 ${basez}" rpy="0 0 0"/>
+            <origin xyz="0 0 ${0.5 * lid_length}" rpy="0 0 0"/>
             <geometry>
-                <box size="${palm_length} ${defwidth} ${defwidth}"/>
+                <<cylinder radius="${lid_radius}" length="${lid_length}"/>
             </geometry>
         </visual>
         <inertial>
-            <origin xyz="0 0 0" rpy="0 0 0"/>
-            <mass value="${0.01 * palm_length}"/>
+            <origin xyz="0 0 ${0.5 * lid_length}" rpy="0 0 0"/>
+            <mass value="0.01"/>
             <inertia
                 ixx="0.0" ixy="0.0" ixz="0.0"
@@ -26,4 +26,18 @@
                 izz="${(0.015 * palm_length * palm_length)/12}"/>
         </inertial>
+    </link>
+    <link name="lidar_base">
+        <collision>
+            <origin xyz="0 0 ${1.5 * lid_length}" rpy="0 0 0"/>
+            <geometry>
+                <<cylinder radius="${lid_radius}" length="0.07357"/>
+            </geometry>
+        </collision>
+        <visual>
+            <origin xyz="0 0 ${1.5 * lid_length}" rpy="0 0 0"/>
+            <geometry>
+                <<cylinder radius="${lid_radius}" length="0.07357"/>
+            </geometry>
+        </visual>
     </link>
     <!-- descripcion de los joints del gripper-->

File: models/mbzirc/simple_gripper.xacro (robot description, xacro)
@@ -27,5 +27,5 @@
         <inertial>
             <origin xyz="0 0 0" rpy="0 0 0"/>
-            <mass value="${0.01 * palm_length}"/>
+            <mass value="${palm_length}"/>
             <inertia
                 ixx="0.0" ixy="0.0" ixz="0.0"
@@ -49,5 +49,5 @@
         <inertial>
             <origin xyz="0 0 0" rpy="0 0 0"/>
-            <mass value="${0.01 * finger_length}"/>
+            <mass value="${finger_length}"/>
             <inertia
                 ixx="${(0.015 * finger_length * finger_length)/12}" ixy="0.0" ixz="0.0"
@@ -71,5 +71,5 @@
         <inertial>
             <origin xyz="0 0 0" rpy="0 ${tip_rot} 0"/>
-            <mass value="${0.01 * tip_length}"/>
+            <mass value="${tip_length}"/>
             <inertia
                 ixx="${(0.015 * tip_length * tip_length)/12}" ixy="0.0" ixz="0.0"
@@ -93,5 +93,5 @@
         <inertial>
             <origin xyz="0 0 0" rpy="0 0 0"/>
-            <mass value="${0.01 * finger_length}"/>
+            <mass value="${0finger_length}"/>
             <inertia
                 ixx="${(0.015 * finger_length * finger_length)/12}" ixy="0.0" ixz="0.0"
@@ -115,5 +115,5 @@
         <inertial>
             <origin xyz="0 0 0" rpy="0 ${-tip_rot} 0"/>
-            <mass value="${0.01 * tip_length}"/>
+            <mass value="${tip_length}"/>
             <inertia
                 ixx="${(0.015 * tip_length * tip_length)/12}" ixy="0.0" ixz="0.0"

Commit message: finished lidar model and joints

File: models/mbzirc/lidar.xacro (robot description, xacro)
@@ -7,45 +7,53 @@
     <link name="lidar_base">
         <collision>
-            <origin xyz="0 0 ${0.5 * lid_length}" rpy="0 0 0"/>
+            <origin xyz="0 0 ${0.5 * lid_length + 0.01}" rpy="0 0 0"/>
             <geometry>
-                <<cylinder radius="${lid_radius}" length="${lid_length}"/>
+                <cylinder radius="${lid_radius}" length="${lid_length}"/>
             </geometry>
         </collision>
         <visual>
-            <origin xyz="0 0 ${0.5 * lid_length}" rpy="0 0 0"/>
+            <origin xyz="0 0 ${0.5 * lid_length + 0.01}" rpy="0 0 0"/>
             <geometry>
-                <<cylinder radius="${lid_radius}" length="${lid_length}"/>
+                <cylinder radius="${lid_radius}" length="${lid_length}"/>
             </geometry>
         </visual>
         <inertial>
-            <origin xyz="0 0 ${0.5 * lid_length}" rpy="0 0 0"/>
-            <mass value="0.01"/>
+            <origin xyz="0 0 ${0.5 * lid_length + 0.01}" rpy="0 0 0"/>
+            <mass value="1.2"/>
             <inertia
-                ixx="0.0" ixy="0.0" ixz="0.0"
-                iyy="${(0.015 * palm_length * palm_length)/12}" iyz="0.0"
-                izz="${(0.015 * palm_length * palm_length)/12}"/>
+                ixx="0.001087473" ixy="0.0" ixz="0.0"
+                iyy="0.001087473" iyz="0.0"
+                izz="0.001092437"/>
         </inertial>
     </link>
-    <link name="lidar_base">
+    <link name="lidar_top">
         <collision>
-            <origin xyz="0 0 ${1.5 * lid_length}" rpy="0 0 0"/>
+            <origin xyz="0 0 ${1.5 * lid_length + 0.01}" rpy="0 0 0"/>
             <geometry>
-                <<cylinder radius="${lid_radius}" length="0.07357"/>
+                <cylinder radius="${lid_radius}" length="0.07357"/>
             </geometry>
         </collision>
         <visual>
-            <origin xyz="0 0 ${1.5 * lid_length}" rpy="0 0 0"/>
+            <origin xyz="0 0 ${1.5 * lid_length + 0.01}" rpy="0 0 0"/>
             <geometry>
-                <<cylinder radius="${lid_radius}" length="0.07357"/>
+                <cylinder radius="${lid_radius}" length="0.07357"/>
             </geometry>
         </visual>
+        <inertial>
+            <origin xyz="0 0 ${1.5 * lid_length + 0.01}" rpy="0 0 0"/>
+            <mass value="0.1"/>
+            <inertia
+                ixx="0.000090623" ixy="0.0" ixz="0.0"
+                iyy="0.000090623" iyz="0.0"
+                izz="0.000091036"/>
+        </inertial>
     </link>
     <!-- descripcion de los joints del gripper-->
-     <joint name="left_joint" type="revolute">
-        <parent link="gripper_palm"/>
-        <child link="gripper_left_finger"/>
-        <origin xyz="0.06 0 -0.09" rpy="0 0 0"/>
-            <limit lower="-1" upper="1" effort="10" velocity="3"/>
-            <axis xyz="0 1 0"/>
+     <joint name="lidar_joint" type="revolute">
+        <parent link="lidar_base"/>
+        <child link="lidar_top"/>
+        <origin xyz="0 0 -0.036785" rpy="0 0 0"/>
+            <limit lower="-10000000000000000000" upper="1000000000000000000" effort="10" velocity="3"/>
+            <axis xyz="0 0 1"/>
      </joint>
 </robot>

File: models/mbzirc/model.xacro (robot description, xacro)
@@ -20,7 +20,14 @@
   <xacro:include filename="$(find delivery_uav)/models/mbzirc/simple_gripper.xacro" />
   <!-- Join the uav to the gripper-->
-  <joint name="arm_gripper_joint" type="fixed">
+  <joint name="uav_gripper_joint" type="fixed">
     <parent link="base_link"/>
     <child link="gripper_palm"/>
+  </joint>
+  <!-- Include lidar-->
+  <xacro:include filename="$(find delivery_uav)/models/mbzirc/lidar.xacro" />
+  <!-- Join the uav to the lidar-->
+  <joint name="uav_lidar_joint" type="fixed">
+    <parent link="base_link"/>
+    <child link="lidar_base"/>
   </joint>
   <!-- CAMBIOS FINAL-->

File: models/mbzirc/simple_gripper.xacro (robot description, xacro)
@@ -93,5 +93,5 @@
         <inertial>
             <origin xyz="0 0 0" rpy="0 0 0"/>
-            <mass value="${0finger_length}"/>
+            <mass value="${finger_length}"/>
             <inertia
                 ixx="${(0.015 * finger_length * finger_length)/12}" ixy="0.0" ixz="0.0"
