Commit message: adjusted lidar weights

File: models/mbzirc/lidar_2d.xacro (robot description, xacro)
@@ -20,5 +20,5 @@
         <inertial>
             <origin xyz="0 0 ${0.5 * lid_length + 0.01}" rpy="0 0 0"/>
-            <mass value="1.2"/>
+            <mass value="0.2"/>
             <inertia
                 ixx="0.001087473" ixy="0.0" ixz="0.0"

File: models/mbzirc/lidar_3d.xacro (robot description, xacro)
@@ -20,5 +20,5 @@
         <inertial>
             <origin xyz="0 0 ${0.5 * lid_length + 0.01}" rpy="0 0 0"/>
-            <mass value="1.2"/>
+            <mass value="0.2"/>
             <inertia
                 ixx="0.001087473" ixy="0.0" ixz="0.0"

Commit message: gripper plugin added

File: models/mbzirc/lidar_2d.xacro (robot description, xacro)
@@ -54,5 +54,5 @@
         <child link="lidar_top"/>
         <origin xyz="0 0 -0.036785" rpy="0 0 0"/>
-            <limit lower="-10000000000000000000" upper="1000000000000000000" effort="10" velocity="3"/>
+            <limit lower="0" upper="0.00001" effort="10" velocity="3"/>
             <axis xyz="0 0 1"/>
      </joint>

File: models/mbzirc/simple_gripper.xacro (robot description, xacro)
@@ -49,5 +49,5 @@
         <inertial>
             <origin xyz="0 0 0" rpy="0 0 0"/>
-            <mass value="${finger_length}"/>
+            <mass value="${2 * finger_length}"/>
             <inertia
                 ixx="${(0.015 * finger_length * finger_length)/12}" ixy="0.0" ixz="0.0"
@@ -71,5 +71,5 @@
         <inertial>
             <origin xyz="0 0 0" rpy="0 ${tip_rot} 0"/>
-            <mass value="${tip_length}"/>
+            <mass value="${2 * tip_length}"/>
             <inertia
                 ixx="${(0.015 * tip_length * tip_length)/12}" ixy="0.0" ixz="0.0"
@@ -93,5 +93,5 @@
         <inertial>
             <origin xyz="0 0 0" rpy="0 0 0"/>
-            <mass value="${finger_length}"/>
+            <mass value="${2 * finger_length}"/>
             <inertia
                 ixx="${(0.015 * finger_length * finger_length)/12}" ixy="0.0" ixz="0.0"
@@ -115,5 +115,5 @@
         <inertial>
             <origin xyz="0 0 0" rpy="0 ${-tip_rot} 0"/>
-            <mass value="${tip_length}"/>
+            <mass value="${2 * tip_length}"/>
             <inertia
                 ixx="${(0.015 * tip_length * tip_length)/12}" ixy="0.0" ixz="0.0"
@@ -145,3 +145,15 @@
         <child link="gripper_right_tip"/>
      </joint>
+   <gazebo>
+    <plugin name="gazebo_ros_left_force" filename="libgazebo_ros_force.so">
+      <bodyName>gripper_left_finger</bodyName>
+      <topicName>/uav_left_force</topicName>
+    </plugin>
+  </gazebo>
+  <gazebo>
+    <plugin name="gazebo_ros_right_force" filename="libgazebo_ros_force.so">
+      <bodyName>gripper_right_finger</bodyName>
+      <topicName>/uav_right_force</topicName>
+    </plugin>
+  </gazebo>
 </robot>

Commit message: Trabajo de 7 mayo, mañana - cambiados nombres de launch - añadidas instrucciones a la raiz del proyecto - añadido mesh de hokuyo para el lidar - añadido launch para mundo de pruebas - añadida simulación en RViz Pendiente: Incluir offsets

File: models/mbzirc/lidar_2d.xacro (robot description, xacro)
@@ -37,5 +37,6 @@
             <origin xyz="0 0 ${1.5 * lid_length + 0.01}" rpy="0 0 0"/>
             <geometry>
-                <cylinder radius="${lid_radius}" length="0.07357"/>
+                <!-- <cylinder radius="${lid_radius}" length="0.07357"/> -->
+                <mesh filename="package://delivery_uav/models/mbzirc/meshes/hokuyo.dae"/>
             </geometry>
         </visual>

Commit message: implementado nodo control gripper

File: models/mbzirc/lidar_2d.xacro (robot description, xacro)
@@ -38,5 +38,5 @@
             <geometry>
                 <!-- <cylinder radius="${lid_radius}" length="0.07357"/> -->
-                <mesh filename="package://delivery_uav/models/mbzirc/meshes/hokuyo.dae"/>
+                <mesh filename="package://delivery_uav/models/mbzirc/meshes/hokuyo.dae" scale="1.75 1.75 1.75"/>
             </geometry>
         </visual>
@@ -50,5 +50,5 @@
         </inertial>
     </link>
-    <!-- descripcion de los joints del gripper-->
+    <!-- descripcion de los joints del lidar-->
      <joint name="lidar_joint" type="revolute">
         <parent link="lidar_base"/>
