Commit message: lidar changed to 3d and fixed simulation_lab_offset

File: models/mbzirc/lidar_3d.xacro (robot description, xacro)
@@ -60,5 +60,5 @@
     <sensor type="ray" name="laz">
        <always_on>true</always_on>
-       <pose>0 0 0.117 1.5707 0 0</pose>
+       <pose>0 0 0.117 0 0 0</pose>
        <visualize>true</visualize>
        <update_rate>30</update_rate>
@@ -66,14 +66,14 @@
          <scan>
            <horizontal>
+             <samples>1</samples>
+             <resolution>1</resolution>
+             <min_angle>-0.15</min_angle>
+             <max_angle>0.15</max_angle>
+           </horizontal>
+           <vertical>
              <samples>32</samples>
              <resolution>1</resolution>
              <min_angle>-0.53529248</min_angle>
              <max_angle>0.18622663</max_angle>
-           </horizontal>
-           <vertical>
-             <samples>1</samples>
-             <resolution>1</resolution>
-             <min_angle>-0.15</min_angle>
-             <max_angle>0.15</max_angle>
            </vertical>
          </scan>

File: models/mbzirc/model.xacro (robot description, xacro)
@@ -25,12 +25,16 @@
   </joint>
   <!-- Include lidar-->
-  <xacro:include filename="$(find delivery_uav)/models/mbzirc/lidar_2d.xacro" />
+  <xacro:include filename="$(find velodyne_description)/urdf/VLP-16.urdf.xacro"/>
+  <xacro:VLP-16 parent="base_link" name="uav_ground_truth" topic="/uav_velodyne_points" organize_cloud="false" hz="10" samples="440" gpu="false">
+  <origin xyz="0 0 0.4" rpy="0 0 0"/>
+  </xacro:VLP-16>
+  <!--<xacro:include filename="$(find delivery_uav)/models/mbzirc/lidar_3d.xacro" /> -->
   <!-- Prueba lidar tutorial-->
 <!--   <xacro:include filename="$(find delivery_uav)/models/mbzirc/lidar_2.xacro" /> -->
-  <!-- Join the uav to the lidar-->
+  <!-- Join the uav to the lidar
   <joint name="uav_lidar_joint" type="fixed">
     <parent link="base_link"/>
     <child link="lidar_base"/>
-  </joint>
+  </joint>-->
   <!-- Posicion absoluta para debugging-->
   <xacro:include filename="$(find delivery_uav)/models/mbzirc/absolute_pos.xacro" />

Commit message: Cambiado velodyne por lidar_3d

File: models/mbzirc/lidar_3d.xacro (robot description, xacro)
@@ -61,13 +61,13 @@
        <always_on>true</always_on>
        <pose>0 0 0.117 0 0 0</pose>
-       <visualize>true</visualize>
-       <update_rate>30</update_rate>
+       <visualize>false</visualize>
+       <update_rate>10</update_rate>
        <ray>
          <scan>
            <horizontal>
-             <samples>1</samples>
+             <samples>2000</samples>
              <resolution>1</resolution>
-             <min_angle>-0.15</min_angle>
-             <max_angle>0.15</max_angle>
+             <min_angle>-3.12</min_angle>
+             <max_angle>3.1415</max_angle>
            </horizontal>
            <vertical>
@@ -90,6 +90,7 @@
       </ray>
       <!-- TO DO: probar que el plugin funcione-->
+      <!-- la libreria block laser es la que hace que funcione con pointcloud-->
       <plugin name="gazebo_ros_block_laser_controller" filename="libgazebo_ros_block_laser.so">
-        <topicName>/uav_3d_scan</topicName>
+        <topicName>/uav_laser_scan</topicName>
         <frameName>lidar_top</frameName>
       </plugin>

File: models/mbzirc/model.xacro (robot description, xacro)
@@ -25,16 +25,16 @@
   </joint>
   <!-- Include lidar-->
-  <xacro:include filename="$(find velodyne_description)/urdf/VLP-16.urdf.xacro"/>
+<!--   <xacro:include filename="$(find velodyne_description)/urdf/VLP-16.urdf.xacro"/>
   <xacro:VLP-16 parent="base_link" name="velodyne" topic="/uav_velodyne_points" organize_cloud="false" hz="10" samples="440" gpu="false">
   <origin xyz="0 0 0.4" rpy="0 0 0"/>
-  </xacro:VLP-16>
-  <!--<xacro:include filename="$(find delivery_uav)/models/mbzirc/lidar_3d.xacro" /> -->
+  </xacro:VLP-16> -->
+  <xacro:include filename="$(find delivery_uav)/models/mbzirc/lidar_3d.xacro" />
   <!-- Prueba lidar tutorial-->
 <!--   <xacro:include filename="$(find delivery_uav)/models/mbzirc/lidar_2.xacro" /> -->
-  <!-- Join the uav to the lidar
+<!--   Join the uav to the lidar -->
   <joint name="uav_lidar_joint" type="fixed">
     <parent link="base_link"/>
     <child link="lidar_base"/>
-  </joint>-->
+  </joint>
   <!-- Posicion absoluta para debugging-->
   <xacro:include filename="$(find delivery_uav)/models/mbzirc/absolute_pos.xacro" />

Commit message: Hotfix del lidar

File: models/mbzirc/lidar_3d.xacro (robot description, xacro)
@@ -37,5 +37,6 @@
             <origin xyz="0 0 ${1.5 * lid_length + 0.01}" rpy="0 0 0"/>
             <geometry>
-                <cylinder radius="${lid_radius}" length="0.07357"/>
+                <!-- <cylinder radius="${lid_radius}" length="0.07357"/> -->
+                <mesh filename="package://delivery_uav/models/mbzirc/meshes/hokuyo.dae" scale="1.75 1.75 1.75"/>
             </geometry>
         </visual>
@@ -54,5 +55,5 @@
         <child link="lidar_top"/>
         <origin xyz="0 0 -0.036785" rpy="0 0 0"/>
-            <limit lower="-10000000000000000000" upper="1000000000000000000" effort="10" velocity="3"/>
+            <limit lower="0" upper="0.00001" effort="10" velocity="3"/>
             <axis xyz="0 0 1"/>
      </joint>
@@ -66,5 +67,5 @@
          <scan>
            <horizontal>
-             <samples>2000</samples>
+             <samples>200</samples>
              <resolution>1</resolution>
              <min_angle>-3.12</min_angle>
@@ -72,8 +73,8 @@
            </horizontal>
            <vertical>
-             <samples>32</samples>
+             <samples>20</samples>
              <resolution>1</resolution>
              <min_angle>-0.53529248</min_angle>
-             <max_angle>0.18622663</max_angle>
+             <max_angle>0.53529248</max_angle>
            </vertical>
          </scan>
