Commit message: Cambios en mensajes y nueva pose neutra en gripper

File: models/mbzirc/simple_gripper.xacro (robot description, xacro)
@@ -49,5 +49,5 @@
         <inertial>
             <origin xyz="0 0 0" rpy="0 0 0"/>
-            <mass value="${2 * finger_length}"/>
+            <mass value="${4 * finger_length}"/>
             <inertia
                 ixx="${(0.015 * finger_length * finger_length)/12}" ixy="0.0" ixz="0.0"
@@ -71,5 +71,5 @@
         <inertial>
             <origin xyz="0 0 0" rpy="0 ${tip_rot} 0"/>
-            <mass value="${2 * tip_length}"/>
+            <mass value="${4 * tip_length}"/>
             <inertia
                 ixx="${(0.015 * tip_length * tip_length)/12}" ixy="0.0" ixz="0.0"
@@ -93,5 +93,5 @@
         <inertial>
             <origin xyz="0 0 0" rpy="0 0 0"/>
-            <mass value="${2 * finger_length}"/>
+            <mass value="${4 * finger_length}"/>
             <inertia
                 ixx="${(0.015 * finger_length * finger_length)/12}" ixy="0.0" ixz="0.0"
@@ -115,5 +115,5 @@
         <inertial>
             <origin xyz="0 0 0" rpy="0 ${-tip_rot} 0"/>
-            <mass value="${2 * tip_length}"/>
+            <mass value="${4 * tip_length}"/>
             <inertia
                 ixx="${(0.015 * tip_length * tip_length)/12}" ixy="0.0" ixz="0.0"

Commit message: EDU: central node clean up and path following adjustments

File: models/mbzirc/simple_gripper.xacro (robot description, xacro)
@@ -49,5 +49,5 @@
         <inertial>
             <origin xyz="0 0 0" rpy="0 0 0"/>
-            <mass value="${4 * finger_length}"/>
+            <mass value="${finger_length}"/>
             <inertia
                 ixx="${(0.015 * finger_length * finger_length)/12}" ixy="0.0" ixz="0.0"
@@ -71,5 +71,5 @@
         <inertial>
             <origin xyz="0 0 0" rpy="0 ${tip_rot} 0"/>
-            <mass value="${4 * tip_length}"/>
+            <mass value="${tip_length}"/>
             <inertia
                 ixx="${(0.015 * tip_length * tip_length)/12}" ixy="0.0" ixz="0.0"
@@ -93,5 +93,5 @@
         <inertial>
             <origin xyz="0 0 0" rpy="0 0 0"/>
-            <mass value="${4 * finger_length}"/>
+            <mass value="${finger_length}"/>
             <inertia
                 ixx="${(0.015 * finger_length * finger_length)/12}" ixy="0.0" ixz="0.0"
@@ -115,5 +115,5 @@
         <inertial>
             <origin xyz="0 0 0" rpy="0 ${-tip_rot} 0"/>
-            <mass value="${4 * tip_length}"/>
+            <mass value="${tip_length}"/>
             <inertia
                 ixx="${(0.015 * tip_length * tip_length)/12}" ixy="0.0" ixz="0.0"

Commit message: Added base for gripper experiments

File: models/mbzirc/simple_gripper.xacro (robot description, xacro)
@@ -127,5 +127,5 @@
         <child link="gripper_left_finger"/>
         <origin xyz="0.06 0 -0.09" rpy="0 0 0"/>
-            <limit lower="-1" upper="1" effort="10" velocity="3"/>
+            <limit lower="-1" upper="0.5" effort="10" velocity="3"/>
             <axis xyz="0 1 0"/>
      </joint>
@@ -134,5 +134,5 @@
         <child link="gripper_right_finger"/>
         <origin xyz="-0.06 0 -0.09" rpy="0 0 0"/>
-            <limit lower="-1" upper="1" effort="10" velocity="3"/>
+            <limit lower="-1" upper="0.5" effort="10" velocity="3"/>
             <axis xyz="0 -1 0"/>
      </joint>
@@ -157,3 +157,15 @@
     </plugin>
   </gazebo>
+    <gazebo>
+        <gripper name="gripper_gazebo">
+            <grasp_check>
+                <attach_steps>5</attach_steps>
+                <detach_steps>10</detach_steps>
+                <min_contact_count>1</min_contact_count>
+            </grasp_check>
+            <gripper_link>gripper_left_tip</gripper_link>
+            <gripper_link>gripper_right_tip</gripper_link>
+            <palm_link>gripper_palm</palm_link>
+        </gripper>
+    </gazebo>
 </robot>
