Commit message: Simulación fallida con mis paquetes

File: urdf/lidar.xacro (robot description, xacro)
@@ -5,5 +5,5 @@
     <joint name="hokuyo_joint" type="fixed">
       <axis xyz="0 1 0" />
-      <origin xyz="0 0 0" rpy="0 0 0"/>
+      <origin xyz="0 0 0.1" rpy="0 0 0"/>
       <parent link="base_link"/>
       <child link="hokuyo_link"/>
@@ -12,5 +12,5 @@
     <link name="hokuyo_link">
       <collision>
-        <origin xyz="0 0 0" rpy="0 0 0"/>
+        <origin xyz="0 0 0.1" rpy="0 0 0"/>
         <geometry>
     <box size="0.1 0.1 0.1"/>
